File: H38R00/Design/H38R00.sch (EAGLE design)
At the start: 77 parts, among them P1 HEXABIT_17.32_X2_POWER_ONLY, U1 LM5160DNT, U2 TPS65130RGERT, U3 TPS76433DBVT

Commit message: Arranged most silkscreen Added labels
Parts:
- renumbered SJ1 to J+15, SJ2 to J-15, SJ3 to J5, SJ4 to J3V3
Changed lines of the file:
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@@
 <attribute name="TOLERANCE" value="1%"/>
 </part>
-<part name="SJ3" library="jumper" library_urn="urn:adsk.eagle:library:252" deviceset="SJ" device="" package3d_urn="urn:adsk.eagle:package:15471/1"/>
+<part name="J5" library="jumper" library_urn="urn:adsk.eagle:library:252" deviceset="SJ" device="" package3d_urn="urn:adsk.eagle:package:15471/1"/>
 <part name="FB1" library="Hexabitz" deviceset="FB-0603" device="" value="600 Ohm">
 <attribute name="MFN" value="Murata"/>
@@
 <attribute name="VOLTAGE_RATING" value="50V"/>
 </part>
-<part name="SJ1" library="jumper" library_urn="urn:adsk.eagle:library:252" deviceset="SJ" device="" package3d_urn="urn:adsk.eagle:package:15471/1"/>
+<part name="J+15" library="jumper" library_urn="urn:adsk.eagle:library:252" deviceset="SJ" device="" package3d_urn="urn:adsk.eagle:package:15471/1"/>
 <part name="R19" library="Hexabitz" deviceset="R-0603" device="" value="5.36K">
 <attribute name="MFN" value="Vishay"/>
@@
 <part name="D4" library="Hexabitz" deviceset="VLMTG1300-GS08" device="" value="GREEN"/>
 <part name="AGND10" library="supply1" library_urn="urn:adsk.eagle:library:371" deviceset="AGND" device="" value="GND_ISO"/>
-<part name="SJ2" library="jumper" library_urn="urn:adsk.eagle:library:252" deviceset="SJ" device="" package3d_urn="urn:adsk.eagle:package:15471/1"/>
+<part name="J-15" library="jumper" library_urn="urn:adsk.eagle:library:252" deviceset="SJ" device="" package3d_urn="urn:adsk.eagle:package:15471/1"/>
 <part name="R18" library="Hexabitz" deviceset="R-0603" device="" value="5.36K">
 <attribute name="MFN" value="Vishay"/>
@@
 <part name="+3V3" library="supply1" library_urn="urn:adsk.eagle:library:371" deviceset="+3V3" device=""/>
 <part name="AGND15" library="supply1" library_urn="urn:adsk.eagle:library:371" deviceset="AGND" device="" value="GND_ISO"/>
-<part name="SJ4" library="jumper" library_urn="urn:adsk.eagle:library:252" deviceset="SJ" device="" package3d_urn="urn:adsk.eagle:package:15471/1"/>
+<part name="J3V3" library="jumper" library_urn="urn:adsk.eagle:library:252" deviceset="SJ" device="" package3d_urn="urn:adsk.eagle:package:15471/1"/>
 </parts>
 <sheets>
@@
 <attribute name="TOLERANCE" x="244.8814" y="190.5" size="1.778" layer="96" rot="R90"/>
 </instance>
-<instance part="SJ3" gate="1" x="241.3" y="176.53" smashed="yes" rot="R90">
+<instance part="J5" gate="1" x="241.3" y="176.53" smashed="yes" rot="R90">
 <attribute name="NAME" x="238.76" y="173.99" size="1.778" layer="95" rot="R90"/>
 <attribute name="VALUE" x="245.11" y="173.99" size="1.778" layer="96" rot="R90"/>
@@
 <attribute name="VOLTAGE_RATING" x="170.434" y="104.14" size="1.778" layer="96"/>
 </instance>
-<instance part="SJ1" gate="1" x="227.33" y="127" smashed="yes" rot="R90">
+<instance part="J+15" gate="1" x="227.33" y="127" smashed="yes" rot="R90">
 <attribute name="NAME" x="224.79" y="124.46" size="1.778" layer="95" rot="R90"/>
 <attribute name="VALUE" x="231.14" y="124.46" size="1.778" layer="96" rot="R90"/>
@@
 <attribute name="VALUE" x="255.27" y="130.81" size="1.778" layer="96"/>
 </instance>
-<instance part="SJ2" gate="1" x="227.33" y="58.42" smashed="yes" rot="R90">
+<instance part="J-15" gate="1" x="227.33" y="58.42" smashed="yes" rot="R90">
 <attribute name="NAME" x="224.79" y="55.88" size="1.778" layer="95" rot="R90"/>
 <attribute name="VALUE" x="231.14" y="55.88" size="1.778" layer="96" rot="R90"/>
@@
 <attribute name="VALUE" x="26.67" y="26.67" size="1.778" layer="96"/>
 </instance>
-<instance part="SJ4" gate="1" x="41.91" y="46.99" smashed="yes" rot="R90">
+<instance part="J3V3" gate="1" x="41.91" y="46.99" smashed="yes" rot="R90">
 <attribute name="NAME" x="39.37" y="44.45" size="1.778" layer="95" rot="R90"/>
 <attribute name="VALUE" x="45.72" y="44.45" size="1.778" layer="96" rot="R90"/>
@@
 <pinref part="R20" gate="G$1" pin="2"/>
 <wire x1="241.3" y1="185.42" x2="241.3" y2="181.61" width="0.1524" layer="91"/>
-<pinref part="SJ3" gate="1" pin="2"/>
+<pinref part="J5" gate="1" pin="2"/>
 </segment>
 </net>
@@
 <junction x="241.3" y="170.18"/>
 <wire x1="241.3" y1="171.45" x2="241.3" y2="170.18" width="0.1524" layer="91"/>
-<pinref part="SJ3" gate="1" pin="1"/>
+<pinref part="J5" gate="1" pin="1"/>
 <pinref part="P+2" gate="1" pin="+5V"/>
 <wire x1="250.19" y1="179.07" x2="250.19" y2="170.18" width="0.1524" layer="91"/>
@@
 <pinref part="P+4" gate="1" pin="+5V"/>
 <wire x1="41.91" y1="54.61" x2="41.91" y2="52.07" width="0.1524" layer="91"/>
-<pinref part="SJ4" gate="1" pin="2"/>
+<pinref part="J3V3" gate="1" pin="2"/>
 </segment>
 </net>
@@
 <wire x1="240.03" y1="110.49" x2="240.03" y2="114.3" width="0.1524" layer="91"/>
 <junction x="240.03" y="114.3"/>
-<pinref part="SJ1" gate="1" pin="1"/>
+<pinref part="J+15" gate="1" pin="1"/>
 <wire x1="227.33" y1="121.92" x2="227.33" y2="114.3" width="0.1524" layer="91"/>
 </segment>
@@
 <wire x1="227.33" y1="73.66" x2="227.33" y2="71.12" width="0.1524" layer="91"/>
 <junction x="227.33" y="71.12"/>
-<pinref part="SJ2" gate="1" pin="2"/>
+<pinref part="J-15" gate="1" pin="2"/>
 <wire x1="227.33" y1="63.5" x2="227.33" y2="71.12" width="0.1524" layer="91"/>
 </segment>
@@
 <net name="N$31" class="0">
 <segment>
-<pinref part="SJ1" gate="1" pin="2"/>
+<pinref part="J+15" gate="1" pin="2"/>
 <pinref part="R19" gate="G$1" pin="1"/>
 <wire x1="227.33" y1="132.08" x2="227.33" y2="137.16" width="0.1524" layer="91"/>
@@
 <net name="N$33" class="0">
 <segment>
-<pinref part="SJ2" gate="1" pin="1"/>
+<pinref part="J-15" gate="1" pin="1"/>
 <pinref part="R18" gate="G$1" pin="1"/>
 <wire x1="227.33" y1="53.34" x2="227.33" y2="41.91" width="0.1524" layer="91"/>
@@
 <junction x="41.91" y="38.1"/>
 <wire x1="41.91" y1="41.91" x2="41.91" y2="38.1" width="0.1524" layer="91"/>
-<pinref part="SJ4" gate="1" pin="1"/>
+<pinref part="J3V3" gate="1" pin="1"/>
 </segment>
 </net>

Commit message: Finished arranging silkscreen Added polygons and isolation barrier
Connections:
- net AGND renamed IGND
Changed lines of the file:
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@@
 </segment>
 </net>
-<net name="AGND" class="0">
+<net name="IGND" class="0">
 <segment>
 <pinref part="C20" gate="G$1" pin="2"/>
@@
 <wire x1="31.75" y1="78.74" x2="31.75" y2="83.82" width="0.1524" layer="91"/>
 <wire x1="31.75" y1="83.82" x2="27.94" y2="83.82" width="0.1524" layer="91"/>
-<pinref part="P1" gate="G$1" pin="GND2"/>
-<wire x1="27.94" y1="78.74" x2="31.75" y2="78.74" width="0.1524" layer="91"/>
-<junction x="31.75" y="78.74"/>
 <pinref part="P1" gate="G$1" pin="GND9"/>
 <wire x1="27.94" y1="43.18" x2="31.75" y2="43.18" width="0.1524" layer="91"/>
@@
 <wire x1="27.94" y1="38.1" x2="31.75" y2="38.1" width="0.1524" layer="91"/>
 <junction x="31.75" y="38.1"/>
+<pinref part="P1" gate="G$1" pin="GND2"/>
+<wire x1="27.94" y1="78.74" x2="31.75" y2="78.74" width="0.1524" layer="91"/>
+<junction x="31.75" y="78.74"/>
 </segment>
 </net>
@@
 <segment>
 <pinref part="+3V3" gate="G$1" pin="+3V3"/>
-<pinref part="P1" gate="G$1" pin="VDD2"/>
 <wire x1="31.75" y1="149.86" x2="31.75" y2="139.7" width="0.1524" layer="91"/>
-<wire x1="31.75" y1="139.7" x2="31.75" y2="134.62" width="0.1524" layer="91"/>
-<wire x1="31.75" y1="134.62" x2="27.94" y2="134.62" width="0.1524" layer="91"/>
 <pinref part="P1" gate="G$1" pin="VDD1"/>
 <wire x1="27.94" y1="139.7" x2="31.75" y2="139.7" width="0.1524" layer="91"/>
@@
 <wire x1="27.94" y1="93.98" x2="31.75" y2="93.98" width="0.1524" layer="91"/>
 <wire x1="31.75" y1="93.98" x2="31.75" y2="99.06" width="0.1524" layer="91"/>
-<junction x="31.75" y="134.62"/>
 <pinref part="P1" gate="G$1" pin="VDD9"/>
 <wire x1="31.75" y1="99.06" x2="31.75" y2="134.62" width="0.1524" layer="91"/>
+<wire x1="31.75" y1="134.62" x2="31.75" y2="139.7" width="0.1524" layer="91"/>
 <wire x1="27.94" y1="99.06" x2="31.75" y2="99.06" width="0.1524" layer="91"/>
 <junction x="31.75" y="99.06"/>
-</segment>
-</net>
+<pinref part="P1" gate="G$1" pin="VDD2"/>
+<wire x1="27.94" y1="134.62" x2="31.75" y2="134.62" width="0.1524" layer="91"/>
+<junction x="31.75" y="134.62"/>
+</segment>
+</net>
