File: H38R00/Design/H38R00.sch (EAGLE design)
At the start: 77 parts, among them P1 HEXABIT_17.32_X2_POWER_ONLY, U1 LM5160DNT, U2 TPS65130RGERT, U3 TPS76433DBVT

Commit message: Adding BOM Updating some params Ready for release Rev0
Parts:
- C25, C26, C27, C28, C32: OCTOPART_URL (none) -> https://octopart.com/grm21bc71e106ke11l-murata-51454492?r=s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; OCTOPAR_URL https://octopart.com/grm21bc71e106ke11l-murata-51454492?r=s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 -> (none)
- C29, C3: OCTOPART_URL (none) -> https://octopart.com/885012207026-w%C3%BCrth+elektronik-654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; OCTOPAR_URL https://octopart.com/885012207026-w%C3%BCrth+elektronik-654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 -> (none)
Changed lines of the file:
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@@
 <attribute name="MFN" value="Würth Elektronik"/>
 <attribute name="MPN" value="885012207026"/>
-<attribute name="OCTOPAR_URL" value="https://octopart.com/885012207026-w%C3%BCrth+elektronik-65419800?r=sp&amp;s=PJ8-ZxRrRL-RXf1D2e7V7w"/>
+<attribute name="OCTOPART_URL" value="https://octopart.com/885012207026-w%C3%BCrth+elektronik-65419800?r=sp&amp;s=PJ8-ZxRrRL-RXf1D2e7V7w"/>
 <attribute name="TOLERANCE" value="10%"/>
 <attribute name="VOLTAGE_RATING" value="10V"/>
@@
 <attribute name="MFN" value="Würth Elektronik"/>
 <attribute name="MPN" value="885012207026"/>
-<attribute name="OCTOPAR_URL" value="https://octopart.com/885012207026-w%C3%BCrth+elektronik-65419800?r=sp&amp;s=PJ8-ZxRrRL-RXf1D2e7V7w"/>
+<attribute name="OCTOPART_URL" value="https://octopart.com/885012207026-w%C3%BCrth+elektronik-65419800?r=sp&amp;s=PJ8-ZxRrRL-RXf1D2e7V7w
+"/>
 <attribute name="TOLERANCE" value="10%"/>
 <attribute name="VOLTAGE_RATING" value="10V"/>
@@
 <attribute name="MFN" value="Murata"/>
 <attribute name="MPN" value="GRM21BC71E106KE11L"/>
-<attribute name="OCTOPAR_URL" value="https://octopart.com/grm21bc71e106ke11l-murata-51454492?r=sp&amp;s=2Vde2RpCRyqy5YYMvYke3Q"/>
+<attribute name="OCTOPART_URL" value="https://octopart.com/grm21bc71e106ke11l-murata-51454492?r=sp&amp;s=2Vde2RpCRyqy5YYMvYke3Q
+"/>
 <attribute name="TOLERANCE" value="10%"/>
 <attribute name="VOLTAGE_RATING" value="25V"/>
@@
 <attribute name="MFN" value="Murata"/>
 <attribute name="MPN" value="GRM21BC71E106KE11L"/>
-<attribute name="OCTOPAR_URL" value="https://octopart.com/grm21bc71e106ke11l-murata-51454492?r=sp&amp;s=2Vde2RpCRyqy5YYMvYke3Q"/>
+<attribute name="OCTOPART_URL" value="https://octopart.com/grm21bc71e106ke11l-murata-51454492?r=sp&amp;s=2Vde2RpCRyqy5YYMvYke3Q
+"/>
 <attribute name="TOLERANCE" value="10%"/>
 <attribute name="VOLTAGE_RATING" value="25V"/>
@@
 <attribute name="MFN" value="Murata"/>
 <attribute name="MPN" value="GRM21BC71E106KE11L"/>
-<attribute name="OCTOPAR_URL" value="https://octopart.com/grm21bc71e106ke11l-murata-51454492?r=sp&amp;s=2Vde2RpCRyqy5YYMvYke3Q"/>
+<attribute name="OCTOPART_URL" value="https://octopart.com/grm21bc71e106ke11l-murata-51454492?r=sp&amp;s=2Vde2RpCRyqy5YYMvYke3Q
+"/>
 <attribute name="TOLERANCE" value="10%"/>
 <attribute name="VOLTAGE_RATING" value="25V"/>
@@
 <attribute name="MFN" value="Murata"/>
 <attribute name="MPN" value="GRM21BC71E106KE11L"/>
-<attribute name="OCTOPAR_URL" value="https://octopart.com/grm21bc71e106ke11l-murata-51454492?r=sp&amp;s=2Vde2RpCRyqy5YYMvYke3Q"/>
+<attribute name="OCTOPART_URL" value="https://octopart.com/grm21bc71e106ke11l-murata-51454492?r=sp&amp;s=2Vde2RpCRyqy5YYMvYke3Q"/>
 <attribute name="TOLERANCE" value="10%"/>
 <attribute name="VOLTAGE_RATING" value="25V"/>
@@
 <attribute name="MFN" value="Murata"/>
 <attribute name="MPN" value="GRM21BC71E106KE11L"/>
-<attribute name="OCTOPAR_URL" value="https://octopart.com/grm21bc71e106ke11l-murata-51454492?r=sp&amp;s=2Vde2RpCRyqy5YYMvYke3Q"/>
-<attribute name="TOLERANCE" value="10%"/>
-<attribute name="VOLTAGE_RATING" value="25V"/>
+<attribute name="OCTOPART_URL" value="https://octopart.com/grm21bc71e106ke11l-murata-51454492?r=sp&amp;s=2Vde2RpCRyqy5YYMvYke3Q"/>
+<attribute name="TOLERANCE" value="10%"/>
+<attribute name="VOLTAGE_RATING" value="25V"/>
